File: UINIO-USB-UART.kicad_sch (KiCad schematic)
At the start: 32 parts, among them J1 Conn_01x07_Male, J2 Conn_01x04_Male, J3 Conn_01x06_Male, J4 Conn_01x06_Male, J5 Conn_01x04_Male, J6 Conn_01x06_Male, SW1 TP-33103, U1 CP2102, U2 CH343P

Commit message: Update PCB.
Parts:
- removed J1: Conn_01x07_Male, Connector_PinHeader_2.54mm:PinHeader_1x07_P2.54mm_Vertical, symbol Connector:Conn_01x07_Male
- removed J3, J6: Conn_01x06_Male, Connector_PinHeader_2.54mm:PinHeader_1x06_P2.54mm_Vertical, symbol Connector:Conn_01x06_Male
- added J1: Conn_01x08_Male, Connector_PinHeader_2.54mm:PinHeader_1x08_P2.54mm_Vertical, symbol Connector:Conn_01x08_Male
- added J3, J6: Conn_01x07_Male, Connector_PinHeader_2.54mm:PinHeader_1x07_P2.54mm_Vertical, symbol Connector:Conn_01x07_Male
Connections:
- net VIO is gone; now on net CH343_VIO: C7.1, U2.1 (VIO)
- net CH343_CTS: now also J6.3 (Pin_3)
- net CH343_RTS: now also J6.4 (Pin_4)
- net CH343_RXD: now also J6.6 (Pin_6)
- net CH343_TXD: now also J6.7 (Pin_7)
- net CH343_VDD_3.3V: now also J6.1 (Pin_1)
- net CH343_VDD_5V: no longer USB1.A4B9 (VBUS)
- net CP2102_*SUSPEND: now also J1.8 (Pin_8)
- net CP2102_CTS: now also J3.3 (Pin_3)
- net CP2102_DCD: now also J1.5 (Pin_5)
- net CP2102_DSR: now also J1.3 (Pin_3)
- net CP2102_DTR: now also J1.4 (Pin_4)
- net CP2102_RI: now also J3.5 (Pin_5)
- net CP2102_RST: now also J1.6 (Pin_6)
- net CP2102_RTS: now also J3.4 (Pin_4)
- net CP2102_RXD: now also J3.6 (Pin_6)
- net CP2102_SUSPEND: now also J1.7 (Pin_7)
- net CP2102_TXD: now also J3.7 (Pin_7)
- net CP2102_VDD_3.3V: now also J3.1 (Pin_1)
- net CP2102_VDD_5V: now also J1.1 (Pin_1)
- net GND: now also J1.2 (Pin_2), J3.2 (Pin_2), J6.2 (Pin_2)
- net at F1.1, USB1.B4A9 (VBUS): now also USB1.A4B9 (VBUS)
- net RI renamed CH343_RI
- net CH343_RI: now also J6.5 (Pin_5)

Commit message: Complete the wiring.
Changed lines of the file:
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@@
   (junction (at 270.51 128.27) (diameter 0) (color 0 0 0 0)
+  )
+  (junction (at 213.36 135.89) (diameter 0) (color 0 0 0 0)
   )
   (junction (at 50.8 123.19) (diameter 0) (color 0 0 0 0)
@@
     (stroke (width 0) (type default) (color 0 0 0 0))
   )
+  (wire (pts (xy 220.98 133.35) (xy 245.11 133.35))
+    (stroke (width 0) (type default) (color 0 0 0 0))
+  )
   (wire (pts (xy 58.42 44.45) (xy 58.42 59.69))
     (stroke (width 0) (type default) (color 0 0 0 0))
@@
     (stroke (width 0) (type default) (color 0 0 0 0))
   )
-  (wire (pts (xy 214.63 135.89) (xy 208.28 135.89))
+  (wire (pts (xy 214.63 135.89) (xy 213.36 135.89))
     (stroke (width 0) (type default) (color 0 0 0 0))
   )
@@
     (stroke (width 0) (type default) (color 0 0 0 0))
   )
-  (wire (pts (xy 220.98 133.35) (xy 245.11 133.35))
-    (stroke (width 0) (type default) (color 0 0 0 0))
-  )
   (wire (pts (xy 128.27 58.42) (xy 153.67 58.42))
     (stroke (width 0) (type default) (color 0 0 0 0))
@@
     (stroke (width 0) (type default) (color 0 0 0 0))
   )
-  (wire (pts (xy 245.11 128.27) (xy 223.52 128.27))
+  (wire (pts (xy 245.11 128.27) (xy 224.79 128.27))
     (stroke (width 0.254) (type default) (color 0 0 0 0))
   )
@@
     (stroke (width 0) (type default) (color 0 0 0 0))
   )
-  (wire (pts (xy 245.11 125.73) (xy 223.52 125.73))
+  (wire (pts (xy 245.11 125.73) (xy 224.79 125.73))
     (stroke (width 0.254) (type default) (color 0 0 0 0))
   )
@@
     (stroke (width 0) (type default) (color 0 0 0 0))
   )
+  (wire (pts (xy 213.36 120.65) (xy 213.36 135.89))
+    (stroke (width 0) (type default) (color 0 0 0 0))
+  )
   (wire (pts (xy 220.98 118.11) (xy 245.11 118.11))
     (stroke (width 0) (type default) (color 0 0 0 0))
@@
     (stroke (width 0) (type default) (color 0 0 0 0))
   )
-  (wire (pts (xy 238.76 120.65) (xy 245.11 120.65))
-    (stroke (width 0) (type default) (color 0 0 0 0))
-  )
   (wire (pts (xy 50.8 110.49) (xy 60.96 110.49))
     (stroke (width 0) (type default) (color 0 0 0 0))
@@
     (stroke (width 0.254) (type default) (color 0 0 0 0))
   )
+  (wire (pts (xy 213.36 120.65) (xy 245.11 120.65))
+    (stroke (width 0) (type default) (color 0 0 0 0))
+  )
   (wire (pts (xy 29.21 139.7) (xy 29.21 140.97))
     (stroke (width 0) (type default) (color 0 0 0 0))
@@
   )
   (wire (pts (xy 167.64 48.26) (xy 167.64 45.72))
+    (stroke (width 0) (type default) (color 0 0 0 0))
+  )
+  (wire (pts (xy 213.36 135.89) (xy 208.28 135.89))
     (stroke (width 0) (type default) (color 0 0 0 0))
   )
@@
     (effects (font (size 1.27 1.27)) (justify right bottom))
   )
-  (label "CP2102_USB_Data_P" (at 223.52 125.73 0)
+  (label "CP2102_USB_Data_P" (at 224.79 125.73 0)
     (effects (font (size 1.27 1.27)) (justify left bottom))
   )
@@
     (effects (font (size 1.27 1.27)) (justify right bottom))
   )
-  (label "CP2102_VDD_5V" (at 238.76 120.65 180)
-    (effects (font (size 1.27 1.27)) (justify right bottom))
-  )
   (label "CP2102_TXD" (at 109.22 143.51 0)
     (effects (font (size 1.27 1.27)) (justify left bottom))
@@
     (effects (font (size 1.27 1.27)) (justify right bottom))
   )
-  (label "CP2102_USB_Data_N" (at 223.52 128.27 0)
-    (effects (font (size 1.27 1.27)) (justify left bottom))
-  )
+  (label "CP2102_USB_Data_N" (at 224.79 128.27 0)
+    (effects (font (size 1.27 1.27)) (justify left bottom))
+  )

Commit message: Generate all of Gerber files.
Connections:
- net CP2102_VDD_5V: no longer USB2.A4B9 (VBUS)
- net at F2.1, USB2.B4A9 (VBUS): now also USB2.A4B9 (VBUS)
Other:
- moved on the sheet: F1
Changed lines of the file:
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@@
     (company "电子技术博客 UinIO.com")
   )
-  (junction (at 58.42 59.69) (diameter 0) (color 0 0 0 0)
-  )
   (junction (at 148.59 53.34) (diameter 0) (color 0 0 0 0)
   )
+  (junction (at 50.8 41.91) (diameter 0) (color 0 0 0 0)
+  )
   (junction (at 29.21 130.81) (diameter 0) (color 0 0 0 0)
   )
@@
   (junction (at 63.5 130.81) (diameter 0) (color 0 0 0 0)
   )
+  (junction (at 223.52 135.89) (diameter 0) (color 0 0 0 0)
+  )
   (junction (at 208.28 135.89) (diameter 0) (color 0 0 0 0)
   )
@@
   (junction (at 128.27 58.42) (diameter 0) (color 0 0 0 0)
   )
+  (junction (at 53.34 59.69) (diameter 0) (color 0 0 0 0)
+  )
   (junction (at 72.39 59.69) (diameter 0) (color 0 0 0 0)
   )
@@
   (junction (at 270.51 128.27) (diameter 0) (color 0 0 0 0)
   )
-  (junction (at 213.36 135.89) (diameter 0) (color 0 0 0 0)
-  )
   (junction (at 50.8 123.19) (diameter 0) (color 0 0 0 0)
   )
   (junction (at 270.51 130.81) (diameter 0) (color 0 0 0 0)
-  )
-  (junction (at 52.07 41.91) (diameter 0) (color 0 0 0 0)
   )
   (no_connect (at 245.11 138.43))
@@
     (stroke (width 0) (type default) (color 0 0 0 0))
   )
-  (wire (pts (xy 58.42 44.45) (xy 58.42 59.69))
-    (stroke (width 0) (type default) (color 0 0 0 0))
-  )
-  (wire (pts (xy 222.25 135.89) (xy 241.3 135.89))
-    (stroke (width 0) (type default) (color 0 0 0 0))
-  )
-  (wire (pts (xy 44.45 59.69) (xy 39.37 59.69))
+  (wire (pts (xy 53.34 44.45) (xy 53.34 59.69))
+    (stroke (width 0) (type default) (color 0 0 0 0))
+  )
+  (wire (pts (xy 222.25 135.89) (xy 223.52 135.89))
+    (stroke (width 0) (type default) (color 0 0 0 0))
+  )
+  (wire (pts (xy 41.91 59.69) (xy 39.37 59.69))
     (stroke (width 0) (type default) (color 0 0 0 0))
   )
@@
     (stroke (width 0) (type default) (color 0 0 0 0))
   )
-  (wire (pts (xy 52.07 38.1) (xy 52.07 41.91))
+  (wire (pts (xy 50.8 38.1) (xy 50.8 41.91))
     (stroke (width 0) (type default) (color 0 0 0 0))
   )
@@
     (stroke (width 0) (type default) (color 0 0 0 0))
   )
-  (wire (pts (xy 214.63 135.89) (xy 213.36 135.89))
-    (stroke (width 0) (type default) (color 0 0 0 0))
-  )
-  (wire (pts (xy 58.42 59.69) (xy 72.39 59.69))
+  (wire (pts (xy 208.28 135.89) (xy 214.63 135.89))
     (stroke (width 0) (type default) (color 0 0 0 0))
   )
@@
     (stroke (width 0) (type default) (color 0 0 0 0))
   )
-  (wire (pts (xy 52.07 41.91) (xy 52.07 57.15))
+  (wire (pts (xy 50.8 41.91) (xy 50.8 57.15))
     (stroke (width 0) (type default) (color 0 0 0 0))
   )
@@
     (stroke (width 0.254) (type default) (color 0 0 0 0))
   )
-  (wire (pts (xy 58.42 44.45) (xy 76.2 44.45))
+  (wire (pts (xy 53.34 44.45) (xy 76.2 44.45))
     (stroke (width 0) (type default) (color 0 0 0 0))
   )
@@
     (stroke (width 0) (type default) (color 0 0 0 0))
   )
-  (wire (pts (xy 52.07 57.15) (xy 76.2 57.15))
+  (wire (pts (xy 50.8 57.15) (xy 76.2 57.15))
     (stroke (width 0) (type default) (color 0 0 0 0))
   )
@@
     (stroke (width 0) (type default) (color 0 0 0 0))
   )
-  (wire (pts (xy 213.36 120.65) (xy 213.36 135.89))
+  (wire (pts (xy 223.52 120.65) (xy 223.52 135.89))
     (stroke (width 0) (type default) (color 0 0 0 0))
   )
@@
     (stroke (width 0) (type default) (color 0 0 0 0))
   )
-  (wire (pts (xy 52.07 41.91) (xy 67.31 41.91))
-    (stroke (width 0) (type default) (color 0 0 0 0))
-  )
   (wire (pts (xy 50.8 120.65) (xy 50.8 123.19))
     (stroke (width 0) (type default) (color 0 0 0 0))
@@
     (stroke (width 0.254) (type default) (color 0 0 0 0))
   )
-  (wire (pts (xy 213.36 120.65) (xy 245.11 120.65))
+  (wire (pts (xy 223.52 120.65) (xy 245.11 120.65))
     (stroke (width 0) (type default) (color 0 0 0 0))
   )
@@
     (stroke (width 0) (type default) (color 0 0 0 0))
   )
-  (wire (pts (xy 213.36 135.89) (xy 208.28 135.89))
+  (wire (pts (xy 53.34 59.69) (xy 72.39 59.69))
     (stroke (width 0) (type default) (color 0 0 0 0))
   )
@@
     (stroke (width 0) (type default) (color 0 0 0 0))
   )
-  (wire (pts (xy 52.07 59.69) (xy 58.42 59.69))
+  (wire (pts (xy 50.8 41.91) (xy 67.31 41.91))
     (stroke (width 0) (type default) (color 0 0 0 0))
   )
@@
     (stroke (width 0) (type default) (color 0 0 0 0))
   )
+  (wire (pts (xy 49.53 59.69) (xy 53.34 59.69))
+    (stroke (width 0) (type default) (color 0 0 0 0))
+  )
   (polyline (pts (xy 16.51 102.87) (xy 16.51 194.31))
     (stroke (width 0) (type default) (color 0 0 0 0))
@@
   )
   (wire (pts (xy 128.27 74.93) (xy 128.27 73.66))
+    (stroke (width 0) (type default) (color 0 0 0 0))
+  )
+  (wire (pts (xy 223.52 135.89) (xy 241.3 135.89))
     (stroke (width 0) (type default) (color 0 0 0 0))
   )
@@
     (pin "1")
   )
-  (symbol (lib_id "power:GND") (at 52.07 38.1 0) (mirror x) (unit 1)
-    (in_bom yes) (on_board yes)
-    (property "Reference" "#PWR04" (id 0) (at 52.07 31.75 0)
-      (effects (font (size 1.27 1.27)) hide)
-    )
-    (property "Value" "GND" (id 1) (at 54.0512 33.9852 0)
-      (effects (font (size 1.27 1.27)) (justify right))
-    )
-    (property "Footprint" "" (id 2) (at 52.07 38.1 0)
-      (effects (font (size 1.27 1.27)) hide)
-    )
-    (property "Datasheet" "" (id 3) (at 52.07 38.1 0)
+  (symbol (lib_id "power:GND") (at 50.8 38.1 0) (mirror x) (unit 1)
+    (in_bom yes) (on_board yes)
+    (property "Reference" "#PWR04" (id 0) (at 50.8 31.75 0)
+      (effects (font (size 1.27 1.27)) hide)
+    )
+    (property "Value" "GND" (id 1) (at 52.7812 33.9852 0)
+      (effects (font (size 1.27 1.27)) (justify right))
+    )
+    (property "Footprint" "" (id 2) (at 50.8 38.1 0)
+      (effects (font (size 1.27 1.27)) hide)
+    )
+    (property "Datasheet" "" (id 3) (at 50.8 38.1 0)
       (effects (font (size 1.27 1.27)) hide)
     )
@@
     (pin "2")
   )
-  (symbol (lib_id "Device:Polyfuse") (at 48.26 59.69 270) (unit 1)
-    (in_bom yes) (on_board yes)
-    (property "Reference" "F1" (id 0) (at 46.99 57.15 90)
+  (symbol (lib_id "Device:Polyfuse") (at 45.72 59.69 270) (unit 1)
+    (in_bom yes) (on_board yes)
+    (property "Reference" "F1" (id 0) (at 44.45 57.15 90)
       (effects (font (size 1.27 1.27)) (justify left))
     )
-    (property "Value" "Polyfuse" (id 1) (at 44.45 62.23 90)
+    (property "Value" "Polyfuse" (id 1) (at 41.91 62.23 90)
       (effects (font (size 1.27 1.27)) (justify left))
     )
-    (property "Footprint" "Fuse:Fuse_1206_3216Metric" (id 2) (at 43.18 60.96 0)
+    (property "Footprint" "Fuse:Fuse_1206_3216Metric" (id 2) (at 40.64 60.96 0)
       (effects (font (size 1.27 1.27)) (justify left) hide)
     )
-    (property "Datasheet" "~" (id 3) (at 48.26 59.69 0)
-      (effects (font (size 1.27 1.27)) hide)
-    )
+    (property "Datasheet" "~" (id 3) (at 45.72 59.69 0)
+      (effects (font (size 1.27 1.27)) hide)
+    )

Commit message: Update libraries.
Other:
- moved on the sheet: C1, C2, C3, C4, U1
