File: UINIO-USB-UART.kicad_pcb (KiCad board)
At the start: 2 copper layers, 72.2 x 20.5 mm, 34 parts, among them J1 Conn_01x08_Male, J2 Conn_01x04_Male, J3 Conn_01x07_Male, J4 Conn_01x06_Male, J5 Conn_01x04_Male, J6 Conn_01x07_Male, SW1 TP-33103, U1 CP2102, U2 CH343P

Commit message: Generate all of Gerber files.
Connections:
- F2 pad 1: Net-(F2-Pad1) -> Net-(USB2-PadA4B9)
- USB2 pad A4B9: /CP2102_VDD_5V -> Net-(USB2-PadA4B9)
- USB2 pad B4A9: Net-(F2-Pad1) -> Net-(USB2-PadA4B9)
Routing:
- net Net-(USB2-PadA4B9): track 0.00 -> 16.0 mm, vias 0 -> 3
- net Net-(F2-Pad1): track 13.4 -> 0.00 mm, vias 2 -> 0
- net /CP2102_VDD_5V: track 60.6 -> 53.1 mm
- net /CP2102_VDD_3.3V: track 38.3 -> 38.9 mm

Commit message: Update README.md.
Routing:
- net GND: track 228.1 -> 224.2 mm, vias 17 -> 16
- net /CH343_VIO: track 47.4 -> 50.0 mm
- net /CH343_VDD_5V: track 60.6 -> 59.0 mm
- net /CH343_VDD_3.3V: track 38.6 -> 40.0 mm
- net Net-(USB2-PadA4B9): track 16.0 -> 15.1 mm
- net /CH343_TXD: track 32.9 -> 33.7 mm

Commit message: Update README.md.
Routing:
- net GND: track 224.2 -> 224.8 mm

Commit message: Update libraries.
Parts:
- added Hole1: Hole-1mm, Uinio:Hole-1mm, F.Cu at (126.4, 91.7)
- added Hole2: Hole-1mm, Uinio:Hole-1mm, F.Cu at (126.5, 108.3)
- added Hole3: Hole-1mm, Uinio:Hole-1mm, F.Cu at (156.1, 108.1)
- added Hole4: Hole-1mm, Uinio:Hole-1mm, F.Cu at (156.3, 91.7)
- added Hole5: Hole-1mm, Uinio:Hole-1mm, F.Cu at (165.4, 91.7)
- added Hole6: Hole-1mm, Uinio:Hole-1mm, F.Cu at (165.4, 108.2)
- added Hole7: Hole-1mm, Uinio:Hole-1mm, F.Cu at (194.7, 108.2)
- added Hole8: Hole-1mm, Uinio:Hole-1mm, F.Cu at (194.8, 91.8)
- moved SW1 0.10 mm to (133.5, 107.5)
Routing:
- net GND: track 224.8 -> 211.6 mm, vias 16 -> 8
